File: KiCad/SerialToDmx.kicad_sch (KiCad schematic)
At the start: 39 parts, among them J1 NAC3MPXXA, J10 Conn_01x08_Pin, J11 Conn_01x08_Pin, J2 NAC3MPXXB, J3 NC3FAV, J4 NC3MAV, J5 NC4FAV, J6 Conn_01x08_Socket, J7 Conn_01x08_Socket, J8 Conn_01x08_Pin, J9 Conn_01x08_Pin, U1 XIAO ESP32 C3, U2 ISOM8710DFFR, U3 ISOM8710DFFR, U4 ISOM8710DFFR, U5 THVD1512DGS, U6 SN74LV1T34DBV

Commit message: With Files
Parts:
- removed D1: 1N4005, Diode_SMD:D_0402_1005Metric, symbol Diode:1N4005
- removed J10, J11, J8, J9: Conn_01x08_Pin, Connector_Faston_Custom:Faston_01x08_pin, symbol Connector:Conn_01x08_Pin
- removed J6, J7: Conn_01x08_Socket, Connector_Faston_Custom:Faston_01x08_socket, symbol Connector:Conn_01x08_Socket
- added D1: D, Resistor_SMD:R_0402_1005Metric, symbol Device:D
- added F11: 01110501Z, Custom_Littlefuse:fuseholder_111_501_Part1, symbol Custom_Littlefuse:Fuseholder_111_501_Part1
- added F12: 01110501Z, Custom_Littlefuse:fuseholder_111_501_Part2, symbol Custom_Littlefuse:Fuseholder_111_501_Part2
- added H10, H5, H9: MountingHole, MountingHole:MountingHole_3.2mm_M3, symbol Mechanical:MountingHole
- added H19, H20, H21, H22: MountingHole, Panelization:mouse-bite-2mm-slot, symbol Mechanical:MountingHole
- added H4: MountingHole_Pad, MountingHole:MountingHole_3.2mm_M3_DIN965_Pad, symbol Mechanical:MountingHole_Pad
- added J10, J11, J8, J9: ~, Custom_Connector_Faston:Faston_01x08_pin, symbol Custom_Connector_Faston:Conn_01x08_Faston_Pin
- added J6, J7: ~, Custom_Connector_Faston:Faston_01x08_socket, symbol Custom_Connector_Faston:Conn_01x08_Faston_Socket
- added R5: 10kR, Resistor_SMD:R_0402_1005Metric, symbol Device:R
- added TH1: TMP61-Q1, Resistor_SMD:R_0402_1005Metric, symbol Device:Thermistor_PTC
- added U7: NSM2012, Package_SO:SOIC-8_3.9x4.9mm_P1.27mm, symbol Custom_Novosense:NSM2012-30B5R-DSPR
- added X1, X11, X12, X13, X14, X15, X16, X17, X18, X2, X3, X4, X5, X6, X7, X8, X81, X82, X83, X84, X85, X86, X87, X88, X91, X92, X93, X94, X95, X96, X97, X98: 1217861-1, Custom_Connector_Faston:Faston_01x01_pin, symbol Custom_Connector_Faston:Conn_01x01-Faston_Pin
- added X61, X62, X63, X64, X65, X66, X67, X68, X71, X72, X73, X74, X75, X76, X77, X78: 63994-1, Custom_Connector_Faston:Faston_01x01_socket, symbol Custom_Connector_Faston:Conn_01x01-Faston_Socket
- C1: value 0.1uC -> 100nF; footprint Capacitor_SMD:C_0402_1005Metric -> Capacitor_SMD:C_0402_1005Metric_Pad0.74x0.62mm_HandSolder
- H1: value MountingHole -> MountingHole_Pad; footprint MountingHole:MountingHole_3.2mm_M3 -> MountingHole:MountingHole_3.2mm_M3_DIN965_Pad; symbol Mechanical:MountingHole -> Mechanical:MountingHole_Pad; now left out of the parts list
- H11: renamed from H7; value Mousebite -> MountingHole
- H12: renamed from H8; value Mousebite -> MountingHole
- H13: renamed from H9; value Mousebite -> MountingHole
- H14: renamed from H10; value Mousebite -> MountingHole
- H15: renamed from H11; value Mousebite -> MountingHole
- H16: renamed from H12; value Mousebite -> MountingHole; footprint Panelization:mouse-bite-3.5mm-slot -> Panelization:mouse-bite-2mm-slot
- H17: renamed from H13; value Mousebite -> MountingHole; footprint Panelization:mouse-bite-3.5mm-slot -> Panelization:mouse-bite-2mm-slot
- H18: renamed from H14; value Mousebite -> MountingHole
- H2: renamed from H3; value MountingHole -> MountingHole_Pad; footprint MountingHole:MountingHole_3.2mm_M3 -> MountingHole:MountingHole_3.2mm_M3_DIN965_Pad; symbol Mechanical:MountingHole -> Mechanical:MountingHole_Pad; now left out of the parts list
- H3: renamed from H5; value MountingHole -> MountingHole_Pad; footprint MountingHole:MountingHole_3.2mm_M3 -> MountingHole:MountingHole_3.2mm_M3_DIN965_Pad; symbol Mechanical:MountingHole -> Mechanical:MountingHole_Pad; now left out of the parts list
- H6: renamed from H2; now left out of the parts list
- H7: renamed from H4; now left out of the parts list
- H8: renamed from H6; now left out of the parts list
- J1: footprint NeutrikCustom:NAC3MPXXA -> Custom_Neutrik:NAC3MPXXA
- J2: footprint NeutrikCustom:NAC3MPXXB -> Custom_Neutrik:NAC3MPXXB
- J3: footprint NeutrikCustom:NC3FAV -> Connector_Audio:Jack_XLR_Neutrik_NC3FAV_Vertical
- J4: footprint NeutrikCustom:NC3MAV -> Connector_Audio:Jack_XLR_Neutrik_NC3MAV_Vertical
- J5: footprint NeutrikCustom:NC4FAV -> Connector_Audio:Jack_XLR_Neutrik_NC4FAV_Vertical
- PS1: footprint IRM-45-12:CONV_IRM-45-12 -> Custom_Meanwell:CONV_IRM-45-12
- PS2: footprint CONV_R-78E5.0-0.5:CONV_R-78E5.0-0.5 -> Custom_Recom:CONV_R-78E5.0-0.5
- PS3: footprint TracoCustom:CONV_TEA_1-0505 -> Converter_DCDC:Converter_DCDC_TRACO_TEA1-xxxx_THT
- U2: renamed from U5; footprint TICustom:DGS0010A_N -> Custom_TI:DGS0010A_N
- U3: renamed from U4; footprint TICustom:ISOM8710 -> Custom_TI:ISOM8710
- U4: renamed from U2; footprint TICustom:ISOM8710 -> Custom_TI:ISOM8710
- U5: renamed from U3; footprint TICustom:ISOM8710 -> Custom_TI:ISOM8710
- renumbered R3 to R1, R1 to R3
Connections:
- net 5V: now also D1.2 (A), R5.1, U7.8 (VCC)
- net DMX+: now also X63.1, X73.1
- net DMX-: now also X62.1, X72.1
- net GND: now also H1.1, H2.1, H3.1, H4.1, TH1.2, U7.1 (IP+), U7.2 (IP+), U7.5 (GND), U7.6 (NC), X64.1, X74.1; no longer J5.2
- net GND-Connection-Bridge: now also X14.1, X4.1
- net GND-Connection-In-Termination: now also X84.1
- net GND-Connection-Out-Termination: now also X94.1
- net GND_Iso: now also X61.1, X71.1
- net L: now also F12.2, X65.1, X75.1; no longer PS1.AC/L
- net L-Connection-Bridge: now also X15.1, X5.1
- net L-Connection-Termination: now also X85.1, X86.1
- net L-switched: now also X66.1
- net N: now also X67.1, X77.1
- net N-Connection-Bridge: now also X17.1, X7.1
- net N-Connection-Termination: now also X87.1, X88.1
- net N-switched: now also X68.1
- net at U1.14 (VUSB): now also D1.1 (K)
- net LED-Current-Sensor: now reaches U1.5 (D4)
- net LED-Current-Sensor: now also U7.7 (VIOUT)
- net Temperature Sensor: now reaches U1.6 (D5)
- net Temperature Sensor: now also R5.2, TH1.1
- new net: X13.1, X3.1
- new net: X1.1, X11.1
- new net: X12.1, X2.1
- new net L-Fused: F11.1, PS1.AC/L
- new net LED-GND: J5.2, U7.3 (IP-), U7.4 (IP-)
- no-connect marks 23 -> 21
Other:
- note added: "Diagnostics"
- moved on the sheet: H11, H12, H13, H14, H15, H16, H17, H18, H6, H7, H8, PS1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

Commit message: Switched Female and Male XLR 3-Pin Connectors
Parts:
- added U8: NSM2012-10B5R-DSPR, Package_SO:SOIC-8_3.9x4.9mm_P1.27mm, symbol Custom_Novosense:NSM2012-10B5R-DSPR
- J3: value NC3FAV -> NC3MAV; footprint Connector_Audio:Jack_XLR_Neutrik_NC3FAV_Vertical -> Custom_Neutrik:NC3MAV; symbol Connector_Audio:NC3FAV -> Connector_Audio:NC3MAV
- J4: value NC3MAV -> NC3FAV; footprint Connector_Audio:Jack_XLR_Neutrik_NC3MAV_Vertical -> Custom_Neutrik:NC3FAV; symbol Connector_Audio:NC3MAV -> Connector_Audio:NC3FAV
- J5: footprint Connector_Audio:Jack_XLR_Neutrik_NC4FAV_Vertical -> Custom_Neutrik:NC4FAV
- U7: value NSM2012 -> NSM2012-10B5R-DSPR; symbol Custom_Novosense:NSM2012-30B5R-DSPR -> Custom_Novosense:NSM2012-10B5R-DSPR
Connections:
- net 5V: now also U8.8 (VCC)
- net GND: now also U8.5 (GND), U8.6 (NC); no longer H1.1, H2.1, H3.1, H4.1, J1.G, J2.G, J4.G, J5.1, J5.G, X64.1, X74.1
- net L-Fused: now also U8.1 (IP+), U8.2 (IP+); no longer PS1.AC/L
- net AC-Current-Sensor: now reaches U1.11 (D10)
- net AC-Current-Sensor: now also U8.7 (VIOUT)
- net GND-Connection-Bridge renamed PE-Connection-Bridge
- net GND-Connection-In-Termination renamed PE-Connection-In-Termination
- new net L_Measured: PS1.AC/L, U8.3 (IP-), U8.4 (IP-)
- new net PE: H1.1, H2.1, H3.1, H4.1, J1.G, J2.G, J3.G, J5.1, J5.G, X64.1, X74.1
- no-connect marks 21 -> 20
Other:
- moved on the sheet: F11, F12, PS1, PS2, PS3, R5, TH1
